Commit message: dexnet cylinder panda works

File: franka_description/robots/hand.urdf.xacro (robot description, xacro)
@@ -2,4 +2,4 @@
 <robot xmlns:xacro="http://www.ros.org/wiki/xacro" name="hand">
   <xacro:include filename="hand.xacro"/>
-  <xacro:hand ns="panda" safety_distance="0.03"/>
+  <xacro:hand ns="panda" safety_distance="0"/>
 </robot>

File: franka_description/robots/hand.xacro (robot description, xacro)
@@ -11,4 +11,9 @@
     </xacro:unless>
     <link name="${ns}_hand">
+    <inertial>
+    <origin xyz="0 0 0" rpy="0 0 0"/>
+    <mass value="0.68"/>
+    <inertia ixx="0.1" ixy="0.0" ixz="0.0" iyy="0.1" iyz="0.0" izz="0.1"/>
+</inertial>
       <visual>
         <geometry>
@@ -61,4 +66,9 @@
     </joint>
     <link name="${ns}_leftfinger">
+    <inertial>
+    <origin xyz="0 0 0" rpy="0 0 0"/>
+    <mass value="0.01"/>
+    <inertia ixx="0.1" ixy="0.0" ixz="0.0" iyy="0.1" iyz="0.0" izz="0.1"/>
+</inertial>
       <visual>
         <geometry>
@@ -68,4 +78,9 @@
     </link>
     <link name="${ns}_rightfinger">
+    <inertial>
+    <origin xyz="0 0 0" rpy="0 0 0"/>
+    <mass value="0.01"/>
+    <inertia ixx="0.1" ixy="0.0" ixz="0.0" iyy="0.1" iyz="0.0" izz="0.1"/>
+</inertial>
       <visual>
         <origin xyz="0 0 0" rpy="0 0 ${pi}"/>

File: franka_description/robots/panda_arm.urdf.xacro (robot description, xacro)
@@ -8,11 +8,17 @@
   <xacro:arg name="gazebo" default="false" />
   <xacro:unless value="$(arg gazebo)">
+      <!-- Gazebo requires a joint to a link called "world" for statically mounted robots -->
+  <link name="world"/>
     <!-- Create a URDF for a real hardware -->
     <xacro:include filename="$(find franka_description)/robots/panda_arm.xacro" />
-    <xacro:panda_arm arm_id="$(arg arm_id)" safety_distance="0.03"/>
+    <xacro:panda_arm arm_id="$(arg arm_id)" connected_to="world" safety_distance="0"/>
     <xacro:if value="$(arg hand)">
       <xacro:include filename="$(find franka_description)/robots/hand.xacro"/>
-      <xacro:hand ns="$(arg arm_id)" rpy="0 0 ${-pi/4}" connected_to="$(arg arm_id)_link8" safety_distance="0.03"/>
+      <xacro:hand ns="$(arg arm_id)" rpy="0 0 ${-pi/4}" connected_to="$(arg arm_id)_link8" safety_distance="0"/>
     </xacro:if>
+    <xacro:include filename="$(find franka_description)/robots/panda_arm_gazebo.xacro"/>
+    <xacro:panda_gazebo arm_id="panda"/>
+    <xacro:include filename="$(find franka_description)/robots/panda_control.xacro"/>
+<xacro:panda_control arm_id="panda"/>
   </xacro:unless>
   <xacro:if value="$(arg gazebo)">
@@ -30,5 +36,5 @@
     <!-- Gazebo requires a joint to a link called "world" for statically mounted robots -->
     <link name="world" />
-    <joint name="world_joint" type="fixed">
+    <joint name="virtual_joint" type="fixed">
       <origin xyz="$(arg xyz)" rpy="$(arg rpy)" />
       <parent link="world" />

File: franka_description/robots/panda_arm.xacro (robot description, xacro)
@@ -5,5 +5,5 @@
   <xacro:macro name="panda_arm" params="arm_id:='panda' description_pkg:='franka_description' connected_to:='' xyz:='0 0 0' rpy:='0 0 0' safety_distance:=0">
     <xacro:unless value="${not connected_to}">
-      <joint name="${arm_id}_joint_${connected_to}" type="fixed">
+      <joint name="virtual_joint" type="fixed">
         <parent link="${connected_to}"/>
         <child link="${arm_id}_link0"/>
@@ -12,4 +12,9 @@
     </xacro:unless>
     <link name="${arm_id}_link0">
+      <inertial>
+        <origin xyz="0 0 0" rpy="0 0 0" />
+        <mass value="3.06" />
+        <inertia ixx="0.3" ixy="0.0" ixz="0.0" iyy="0.3" iyz="0.0" izz="0.3" />
+      </inertial>
       <visual>
         <geometry>
@@ -37,4 +42,9 @@
     </link>
     <link name="${arm_id}_link1">
+      <inertial>
+        <origin xyz="0 0 0" rpy="0 0 0" />
+        <mass value="3.06" />
+        <inertia ixx="0.3" ixy="0.0" ixz="0.0" iyy="0.3" iyz="0.0" izz="0.3" />
+      </inertial>
       <visual>
         <geometry>
@@ -62,4 +72,5 @@
     </link>
     <joint name="${arm_id}_joint1" type="revolute">
+    <dynamics damping="1.0"/>
       <safety_controller k_position="100.0" k_velocity="40.0" soft_lower_limit="-2.8973" soft_upper_limit="2.8973"/>
       <origin rpy="0 0 0" xyz="0 0 0.333"/>
@@ -67,7 +78,12 @@
       <child link="${arm_id}_link1"/>
       <axis xyz="0 0 1"/>
-      <limit effort="87" lower="-2.8973" upper="2.8973" velocity="2.1750"/>
+      <limit effort="87" lower="-2.9671" upper="2.9671" velocity="2.3925" />
     </joint>
     <link name="${arm_id}_link2">
+      <inertial>
+      <origin xyz="0 0 0" rpy="0 0 0" />
+      <mass value="3.06" />
+      <inertia ixx="0.3" ixy="0.0" ixz="0.0" iyy="0.3" iyz="0.0" izz="0.3" />
+      </inertial>
       <visual>
         <geometry>
@@ -95,4 +111,5 @@
     </link>
     <joint name="${arm_id}_joint2" type="revolute">
+    <dynamics damping="1.0"/>
       <safety_controller k_position="100.0" k_velocity="40.0" soft_lower_limit="-1.7628" soft_upper_limit="1.7628"/>
       <origin rpy="${-pi/2} 0 0" xyz="0 0 0"/>
@@ -100,7 +117,12 @@
       <child link="${arm_id}_link2"/>
       <axis xyz="0 0 1"/>
-      <limit effort="87" lower="-1.7628" upper="1.7628" velocity="2.1750"/>
+      <limit effort="87" lower="-1.8326" upper="1.8326" velocity="2.3925" />
     </joint>
     <link name="${arm_id}_link3">
+    <inertial>
+    <origin xyz="0 0 0" rpy="0 0 0" />
+    <mass value="3.06" />
+    <inertia ixx="0.3" ixy="0.0" ixz="0.0" iyy="0.3" iyz="0.0" izz="0.3" />
+</inertial>
       <visual>
         <geometry>
@@ -128,4 +150,5 @@
     </link>
     <joint name="${arm_id}_joint3" type="revolute">
+    <dynamics damping="1.0"/>
       <safety_controller k_position="100.0" k_velocity="40.0" soft_lower_limit="-2.8973" soft_upper_limit="2.8973"/>
       <origin rpy="${pi/2} 0 0" xyz="0 -0.316 0"/>
@@ -133,7 +156,12 @@
       <child link="${arm_id}_link3"/>
       <axis xyz="0 0 1"/>
-      <limit effort="87" lower="-2.8973" upper="2.8973" velocity="2.1750"/>
+      <limit effort="87" lower="-2.9671" upper="2.9671" velocity="2.3925" />
     </joint>
     <link name="${arm_id}_link4">
+    <inertial>
+    <origin xyz="0 0 0" rpy="0 0 0" />
+    <mass value="3.06" />
+    <inertia ixx="0.3" ixy="0.0" ixz="0.0" iyy="0.3" iyz="0.0" izz="0.3" />
+</inertial>
       <visual>
         <geometry>
@@ -161,12 +189,18 @@
     </link>
     <joint name="${arm_id}_joint4" type="revolute">
-      <safety_controller k_position="100.0" k_velocity="40.0" soft_lower_limit="-3.0718" soft_upper_limit="-0.0698"/>
+    <dynamics damping="1.0"/>
+      <safety_controller k_position="100.0" k_velocity="40.0" soft_lower_limit="-3.0718" soft_upper_limit="0.0175"/>
       <origin rpy="${pi/2} 0 0" xyz="0.0825 0 0"/>
       <parent link="${arm_id}_link3"/>
       <child link="${arm_id}_link4"/>
       <axis xyz="0 0 1"/>
-      <limit effort="87" lower="-3.0718" upper="-0.0698" velocity="2.1750"/>
+      <limit effort="87" lower="-3.0718" upper="0.0873" velocity="2.1750"/>
     </joint>
     <link name="${arm_id}_link5">
+    <inertial>
+    <origin xyz="0 0 0" rpy="0 0 0" />
+    <mass value="3.06" />
+    <inertia ixx="0.3" ixy="0.0" ixz="0.0" iyy="0.3" iyz="0.0" izz="0.3" />
+</inertial>
       <visual>
         <geometry>
@@ -212,4 +246,5 @@
     </link>
     <joint name="${arm_id}_joint5" type="revolute">
+    <dynamics damping="1.0"/>
       <safety_controller k_position="100.0" k_velocity="40.0" soft_lower_limit="-2.8973" soft_upper_limit="2.8973"/>
       <origin rpy="${-pi/2} 0 0" xyz="-0.0825 0.384 0"/>
@@ -217,7 +252,12 @@
       <child link="${arm_id}_link5"/>
       <axis xyz="0 0 1"/>
-      <limit effort="12" lower="-2.8973" upper="2.8973" velocity="2.6100"/>
+        <limit effort="12" lower="-2.9671" upper="2.9671" velocity="2.8710" />
     </joint>
     <link name="${arm_id}_link6">
+    <inertial>
+    <origin xyz="0 0 0" rpy="0 0 0" />
+    <mass value="3.06" />
+    <inertia ixx="0.3" ixy="0.0" ixz="0.0" iyy="0.3" iyz="0.0" izz="0.3" />
+</inertial>
       <visual>
         <geometry>
@@ -245,4 +285,5 @@
     </link>
     <joint name="${arm_id}_joint6" type="revolute">
+    <dynamics damping="1.0"/>
       <safety_controller k_position="100.0" k_velocity="40.0" soft_lower_limit="-0.0175" soft_upper_limit="3.7525"/>
       <origin rpy="${pi/2} 0 0" xyz="0 0 0"/>
@@ -250,7 +291,12 @@
       <child link="${arm_id}_link6"/>
       <axis xyz="0 0 1"/>
-      <limit effort="12" lower="-0.0175" upper="3.7525" velocity="2.6100"/>
+      <limit effort="12" lower="-0.0873" upper="3.8223" velocity="2.8710" />
     </joint>
     <link name="${arm_id}_link7">
+    <inertial>
+    <origin xyz="0 0 0" rpy="0 0 0" />
+    <mass value="3.06" />
+    <inertia ixx="0.3" ixy="0.0" ixz="0.0" iyy="0.3" iyz="0.0" izz="0.3" />
+</inertial>
       <visual>
         <geometry>
@@ -278,4 +324,5 @@
     </link>
     <joint name="${arm_id}_joint7" type="revolute">
+    <dynamics damping="1.0"/>
       <safety_controller k_position="100.0" k_velocity="40.0" soft_lower_limit="-2.8973" soft_upper_limit="2.8973"/>
       <origin rpy="${pi/2} 0 0" xyz="0.088 0 0"/>
@@ -283,14 +330,19 @@
       <child link="${arm_id}_link7"/>
       <axis xyz="0 0 1"/>
-      <limit effort="12" lower="-2.8973" upper="2.8973" velocity="2.6100"/>
+      <limit effort="12" lower="-2.9671" upper="2.9671" velocity="2.8710" />
     </joint>
     <link name="${arm_id}_link8">
-      <collision>
+    <inertial>
+    <origin xyz="0 0 0" rpy="0 0 0" />
+    <mass value="3.06" />
+    <inertia ixx="0.3" ixy="0.0" ixz="0.0" iyy="0.3" iyz="0.0" izz="0.3" />
+</inertial>
+      <!-- <collision>
         <origin xyz="0.0424 0.0424 -0.0250" rpy="${pi} ${pi/2} ${pi/2}"/>
         <geometry>
           <cylinder radius="${0.03+safety_distance}"  length="0.01" />
         </geometry>
-      </collision>
-      <collision>
+      </collision> -->
+      <!-- <collision>
         <origin xyz="0.0424 0.0424 -0.02" rpy="0 0 0"/>
         <geometry>
@@ -303,5 +355,5 @@
           <sphere radius="${0.03+safety_distance}"  />
         </geometry>
-      </collision>
+      </collision> -->
     </link>
     <joint name="${arm_id}_joint8" type="fixed">
